File: Button PCB/Button PCB.kicad_pcb (KiCad board)
At the start: 2 copper layers, 4 parts

Commit message: Add files via upload
Connections:
- BootButton pad 1: (no net) -> BOOT
- BootButton pad 2: (no net) -> VCC
- BootButton pad 3: (no net) -> GND
- DownButton pad 1: (no net) -> DOWN
- DownButton pad 2: (no net) -> VCC
- DownButton pad 3: (no net) -> GND
- REF** pad 5: (no net) -> BOOT
- REF** pad 6: (no net) -> UP
- REF** pad 7: (no net) -> DOWN
- REF** pad GND: (no net) -> GND
- REF** pad VCC: (no net) -> VCC
- UpButton pad 1: (no net) -> UP
- UpButton pad 2: (no net) -> VCC
- UpButton pad 3: (no net) -> GND
Routing:
- net (no net): track 214.0 -> 0.00 mm
- net VCC: track 0.00 -> 70.6 mm
- net GND: track 0.00 -> 58.0 mm
- net DOWN: track 0.00 -> 50.8 mm
- net UP: track 0.00 -> 27.7 mm
- net BOOT: track 0.00 -> 6.74 mm
Other:
- board outline added: 30 x 65 mm
