File: PCB file/졸작.kicad_sch (KiCad schematic)
At the start: 22 parts, among them SW1 BootButton, SW2 UpButton, SW3 DownButton, U2 DS18B20, U3 DRV8833RTY, U4 MAX1704X

Commit message: Add files via upload
Parts:
- removed PS1: LTC1871(3.3V -> 5V), Converter_DCDC:Converter_DCDC_XP_POWER-ITXxxxxSA_THT, symbol Converter_DCDC:ITX1215SA
- removed U3: DRV8833RTY, Package_DFN_QFN:Texas_RTY_WQFN-16-1EP_4x4mm_P0.65mm_EP2.1x2.1mm_ThermalVias, symbol Driver_Motor:DRV8833RTY
- added BTS7960(MotorDrive): ~, symbol New_Library_symbol_project:BTS7960
- added ChargeModule: ~, symbol New_Library_symbol_project:ChargeModule
- added Converter: ~, symbol New_Library_symbol_project:LM2596Module
- added U1, U3, U5, U6: ~, symbol New_Library_symbol_project:IRL540N
Connections:
- net Battery + is gone; now on net VCC: BT1.1 (+)
- net Battery - is gone; now on net GND: BT1.2 (-)
- net Feltier(+): now also U1. (Gate), U3. (Gate), U5. (Gate)
- net Feltier(-): now also BTS7960(MotorDrive). (Motor(-))
- net GND: now also BTS7960(MotorDrive). (Motor(-)), ChargeModule. (IN+)
- net SCL: now also JP7.1, R9.1, U4.8 (SDA); no longer MPU1.9 (GPIO9), OLED12864I2C1. (SCL)
- net VCC: now also MPU1.5V, BTS7960(MotorDrive). (Motor(-)), ChargeModule. (IN+); no longer MPU1.3.3 (3V3), OLED12864I2C1. (SCL), SW1.1, SW2.1, SW3.1, U2.3 (V_{DD})
- net at MPU1.20 (GPIO20): now also U3. (Gate)
- net at MPU1.10 (GPIO10): now also U1. (Gate)
- net at MPU1.0 (GPIO0): now also BTS7960(MotorDrive). (Motor(-))
- net at MPU1.1 (GPIO1): now also SW3.SH (B)
- net at MPU1.2 (GPIO2): now also SW2.SH (B)
- net at MPU1.21 (GPIO21): now also U5. (Gate)
- net at MPU1.4 (GPIO4): now also U2.2 (DQ)
- net DQ: no longer names the net of MPU1.3 (GPIO3)
- net DQ: now also SW1.SH (B); no longer U2.2 (DQ)
- net GPIO7: no longer names the net of MPU1.7 (GPIO7)
- net GPIO7: now also U6. (Gate); no longer SW3.SH (B)
- net OUT1: no longer names the net of MPU1.5 (GPIO5)
- net OUT1: now also BTS7960(MotorDrive). (Motor(-)); no longer SW1.SH (B)
- net OUT2: no longer names the net of MPU1.6 (GPIO6)
- net OUT2: now also BTS7960(MotorDrive). (Motor(-)); no longer SW2.SH (B)
- removed net SDA: JP7.1, MPU1.8 (GPIO8), OLED12864I2C1. (SCL), R9.1, U4.8 (SDA)
- new net: ChargeModule. (IN+), Converter. (in-) (x2)
- new net: BTS7960(MotorDrive). (Motor(-)), U1. (Gate), U3. (Gate), U5. (Gate)
- new net +12V: BTS7960(MotorDrive). (Motor(-)), Converter. (in-), U6. (Gate)
- new net +3.3V: MPU1.3.3 (3V3), OLED12864I2C1. (SCL), SW1.1, SW2.1, SW3.1, U2.3 (V_{DD})
- new net GNDREF: BTS7960(MotorDrive). (Motor(-)), Converter. (in-)
Other:
- removed sheet Module
- note added: "12V"
- note added: "5V"
- note added: "GND"
- note added: "MAX17043"
- moved on the sheet: BT1, C3, C4, JP3, JP6, JP7, JP8, MPU1, OLED12864I2C1, R10, R11, R12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
